File: PCB1/PCB1a/PCB1a.sch (EAGLE design)
At the start: 24 parts, among them J1 691357310006B, J2 618009231421, J3 ESP32_DEVC_MIN_LEFT, J4 ESP32_DEVC_MIN_RIGHT, U8 74AHCT245, U9 74AHCT245

Commit message: intermediate. commit.
Parts:
- added C1: 470uF, Wurth_Capacitors_WCAP-AS5H:WCAP-AS5H_10X10.5_865230357008
- added C15: 47nF, Wurth_Capacitors_WCAP-CSGP:WCAP-CSGP_0805_H0.8_885012207096_50V(DC)_R
- added C17, C19: 100nF, Wurth_Capacitors_WCAP-CSGP:WCAP-CSGP_0805_H0.8_885012207098_50V(DC)_R
- added C3, C4, C6, C7, C8: 100nF, Discrete:C-0603
- added D1: 5V, Wurth_EMC Components_WE-TVSP:WE-TVSP_DO-214AB_3000W_BI_824551500
- added D11: 24Vdc, Wurth_EMC Components_WE-TVS:WE-TVS_SOT23-3L_824094024
- added R1, R3: 60R, resistor:R-EU_R0805
- added U2: MAX232D, IC:MAX3232-SOIC16
- added U4: TLE9250VSJ, TLE9250VSJ:TLE9250VSJ
Connections:
- removed net CAN_H: J1.6
- removed net CAN_L: J1.5
- removed net N$12: J3.23
- removed net N$18: J4.35
- removed net N$19: J4.32
- removed net N$4: J3.5
- new net +3V3: C19.1, U4.VIO
- new net 232_RX: J2.2, U2.RIN1
- new net 232_TX: J2.3, U2.DOUT1
- new net CAN1_RXD: J4.35, U4.RXD
- new net CAN1_TXD: J3.5, U4.TXD
- new net CAN_N: D11.I/O1, J1.5, R3.2, U4.CANL
- new net CAN_P: D11.I/O2, J1.6, R1.2, U4.CANH
- new net N$20: C15.1, R1.1, R3.1
- new net N$33: C6.2, U2.C1+
- new net N$34: C6.1, U2.C1-
- new net N$35: C7.2, U2.C2+
- new net N$36: C7.1, U2.C2-
- new net N$37: C4.1, U2.V+
- new net N$38: C8.1, U2.V-
- new net N$39: U2.ROUT2
- new net N$40: U2.DIN2
- new net N$46: U2.DOUT2
- new net N$47: U2.RIN2
- new net VCC: C3.1, C4.2, U2.VCC
- net +5V: now also C1.+, C17.1, D1.2, U4.VCC
- net GND: now also C1.-, C15.2, C17.2, C19.2, C3.2, C8.2, D1.1, D11.GND, U2.GND, U4.GND, U4.NEN
- net RX: now also J4.32, U2.ROUT1; no longer J2.2
- net TX: now also J3.23, U2.DIN1; no longer J2.3
Other:
- note added: "Very low electromagnetic emission (EME) allows the use without additional common mode choke TLE9250VSJ"

Commit message: thermals="no"/>
 thermals="no"/>
Changed lines of the file:
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@@
 </plain>
 <instances>
-<instance part="GND1" gate="1" x="12.7" y="12.7" smashed="yes">
-<attribute name="VALUE" x="10.16" y="10.16" size="1.778" layer="96"/>
+<instance part="GND1" gate="1" x="101.6" y="104.14" smashed="yes">
+<attribute name="VALUE" x="99.06" y="101.6" size="1.778" layer="96"/>
 </instance>
 <instance part="HUB75RGB" gate="G$1" x="95.25" y="71.12" smashed="yes" rot="R270">

Commit message: ..
Parts:
- C3, C4, C6, C7, C8: device Discrete:C-0603 -> Wurth_Capacitors_WCAP-CSGP:WCAP-CSGP_0805_H0.8_885012207098_50V(DC)_R
Changed lines of the file:
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@@
 <part name="D11" library="Wurth_EMC Components_WE-TVS" library_urn="urn:adsk.eagle:library:14282971" deviceset="WE-TVS_SOT23-3L_824094024" device="" package3d_urn="urn:adsk.eagle:package:12152380/4" value="24Vdc"/>
 <part name="U2" library="IC" deviceset="MAX3232" device="-SOIC16" value="MAX232D"/>
-<part name="C6" library="Discrete" deviceset="C*" device="-0603" value="100nF"/>
-<part name="C7" library="Discrete" deviceset="C*" device="-0603" value="100nF"/>
-<part name="C3" library="Discrete" deviceset="C*" device="-0603" value="100nF"/>
-<part name="C4" library="Discrete" deviceset="C*" device="-0603" value="100nF"/>
-<part name="C8" library="Discrete" deviceset="C*" device="-0603" value="100nF"/>
+<part name="C6" library="Wurth_Capacitors_WCAP-CSGP" library_urn="urn:adsk.eagle:library:18488985" deviceset="WCAP-CSGP_0805_H0.8" device="_50V(DC)_R" package3d_urn="urn:adsk.eagle:package:18489119/2" technology="_885012207098" value="100nF"/>
+<part name="C7" library="Wurth_Capacitors_WCAP-CSGP" library_urn="urn:adsk.eagle:library:18488985" deviceset="WCAP-CSGP_0805_H0.8" device="_50V(DC)_R" package3d_urn="urn:adsk.eagle:package:18489119/2" technology="_885012207098" value="100nF"/>
+<part name="C3" library="Wurth_Capacitors_WCAP-CSGP" library_urn="urn:adsk.eagle:library:18488985" deviceset="WCAP-CSGP_0805_H0.8" device="_50V(DC)_R" package3d_urn="urn:adsk.eagle:package:18489119/2" technology="_885012207098" value="100nF"/>
+<part name="C4" library="Wurth_Capacitors_WCAP-CSGP" library_urn="urn:adsk.eagle:library:18488985" deviceset="WCAP-CSGP_0805_H0.8" device="_50V(DC)_R" package3d_urn="urn:adsk.eagle:package:18489119/2" technology="_885012207098" value="100nF"/>
+<part name="C8" library="Wurth_Capacitors_WCAP-CSGP" library_urn="urn:adsk.eagle:library:18488985" deviceset="WCAP-CSGP_0805_H0.8" device="_50V(DC)_R" package3d_urn="urn:adsk.eagle:package:18489119/2" technology="_885012207098" value="100nF"/>
 <part name="U$18" library="Power or GND " deviceset="GND_POWER" device=""/>
 <part name="U$19" library="Power or GND " deviceset="GND_POWER" device=""/>
@@
 <attribute name="VALUE" x="48.26" y="72.39" size="1.778" layer="96"/>
 </instance>
-<instance part="C6" gate="C" x="34.29" y="68.58" smashed="yes">
+<instance part="C6" gate="G$1" x="34.29" y="68.58" smashed="yes">
 <attribute name="NAME" x="30.48" y="68.58" size="1.27" layer="95"/>
 <attribute name="VALUE" x="34.29" y="68.58" size="1.27" layer="96"/>
 </instance>
-<instance part="C7" gate="C" x="34.29" y="63.5" smashed="yes">
+<instance part="C7" gate="G$1" x="34.29" y="63.5" smashed="yes">
 <attribute name="NAME" x="30.48" y="63.5" size="1.27" layer="95"/>
 <attribute name="VALUE" x="34.29" y="63.5" size="1.27" layer="96"/>
 </instance>
-<instance part="C3" gate="C" x="82.55" y="68.58" smashed="yes">
+<instance part="C3" gate="G$1" x="82.55" y="68.58" smashed="yes">
 <attribute name="NAME" x="78.74" y="68.58" size="1.27" layer="95"/>
 <attribute name="VALUE" x="82.55" y="68.58" size="1.27" layer="96"/>
 </instance>
-<instance part="C4" gate="C" x="82.55" y="66.04" smashed="yes">
-<attribute name="NAME" x="78.74" y="66.04" size="1.27" layer="95"/>
-<attribute name="VALUE" x="82.55" y="66.04" size="1.27" layer="96"/>
-</instance>
-<instance part="C8" gate="C" x="81.28" y="43.18" smashed="yes">
+<instance part="C4" gate="G$1" x="82.55" y="63.5" smashed="yes">
+<attribute name="NAME" x="78.74" y="63.5" size="1.27" layer="95"/>
+<attribute name="VALUE" x="82.55" y="63.5" size="1.27" layer="96"/>
+</instance>
+<instance part="C8" gate="G$1" x="81.28" y="43.18" smashed="yes">
 <attribute name="NAME" x="77.47" y="43.18" size="1.27" layer="95"/>
 <attribute name="VALUE" x="81.28" y="43.18" size="1.27" layer="96"/>
@@
 <segment>
 <pinref part="U2" gate="G$1" pin="C1+"/>
-<wire x1="43.18" y1="68.58" x2="38.1" y2="68.58" width="0.1524" layer="91"/>
-<pinref part="C6" gate="C" pin="2"/>
+<wire x1="43.18" y1="68.58" x2="39.37" y2="68.58" width="0.1524" layer="91"/>
+<pinref part="C6" gate="G$1" pin="2"/>
 </segment>
 </net>
@@
 <wire x1="43.18" y1="66.04" x2="29.21" y2="66.04" width="0.1524" layer="91"/>
 <wire x1="29.21" y1="66.04" x2="29.21" y2="68.58" width="0.1524" layer="91"/>
-<wire x1="29.21" y1="68.58" x2="30.48" y2="68.58" width="0.1524" layer="91"/>
-<pinref part="C6" gate="C" pin="1"/>
+<wire x1="29.21" y1="68.58" x2="31.75" y2="68.58" width="0.1524" layer="91"/>
+<pinref part="C6" gate="G$1" pin="1"/>
 </segment>
 </net>
@@
 <segment>
 <pinref part="U2" gate="G$1" pin="C2+"/>
-<wire x1="38.1" y1="63.5" x2="43.18" y2="63.5" width="0.1524" layer="91"/>
-<pinref part="C7" gate="C" pin="2"/>
+<wire x1="39.37" y1="63.5" x2="43.18" y2="63.5" width="0.1524" layer="91"/>
+<pinref part="C7" gate="G$1" pin="2"/>
 </segment>
 </net>
@@
 <wire x1="43.18" y1="60.96" x2="29.21" y2="60.96" width="0.1524" layer="91"/>
 <wire x1="29.21" y1="60.96" x2="29.21" y2="63.5" width="0.1524" layer="91"/>
-<wire x1="29.21" y1="63.5" x2="30.48" y2="63.5" width="0.1524" layer="91"/>
-<pinref part="C7" gate="C" pin="1"/>
+<wire x1="29.21" y1="63.5" x2="31.75" y2="63.5" width="0.1524" layer="91"/>
+<pinref part="C7" gate="G$1" pin="1"/>
 </segment>
 </net>
@@
 <segment>
 <pinref part="U2" gate="G$1" pin="V+"/>
-<wire x1="72.39" y1="66.04" x2="78.74" y2="66.04" width="0.1524" layer="91"/>
-<pinref part="C4" gate="C" pin="1"/>
+<wire x1="72.39" y1="66.04" x2="80.01" y2="63.5" width="0.1524" layer="91"/>
+<pinref part="C4" gate="G$1" pin="1"/>
 </segment>
 </net>
 <net name="GND" class="0">
 <segment>
-<wire x1="86.36" y1="68.58" x2="93.98" y2="68.58" width="0.1524" layer="91"/>
+<wire x1="87.63" y1="68.58" x2="93.98" y2="68.58" width="0.1524" layer="91"/>
 <label x="90.17" y="68.58" size="1.27" layer="95"/>
-<pinref part="C3" gate="C" pin="2"/>
+<pinref part="C3" gate="G$1" pin="2"/>
 <pinref part="U$20" gate="G$1" pin="GND"/>
 </segment>
 <segment>
-<wire x1="85.09" y1="43.18" x2="90.17" y2="43.18" width="0.1524" layer="91"/>
+<wire x1="86.36" y1="43.18" x2="90.17" y2="43.18" width="0.1524" layer="91"/>
 <label x="86.36" y="43.18" size="1.27" layer="95"/>
-<pinref part="C8" gate="C" pin="2"/>
+<pinref part="C8" gate="G$1" pin="2"/>
 <pinref part="U$19" gate="G$1" pin="GND"/>
 <wire x1="90.17" y1="40.64" x2="90.17" y2="43.18" width="0.1524" layer="91"/>
@@
 <net name="VCC" class="0">
 <segment>
-<wire x1="86.36" y1="66.04" x2="93.98" y2="66.04" width="0.1524" layer="91"/>
-<label x="90.17" y="66.04" size="1.27" layer="95"/>
-<pinref part="C4" gate="C" pin="2"/>
+<wire x1="87.63" y1="63.5" x2="93.98" y2="63.5" width="0.1524" layer="91"/>
+<label x="90.17" y="63.5" size="1.27" layer="95"/>
+<pinref part="C4" gate="G$1" pin="2"/>
 </segment>
 <segment>
 <pinref part="U2" gate="G$1" pin="VCC"/>
-<wire x1="72.39" y1="68.58" x2="78.74" y2="68.58" width="0.1524" layer="91"/>
+<wire x1="72.39" y1="68.58" x2="80.01" y2="68.58" width="0.1524" layer="91"/>
 <label x="73.66" y="68.58" size="1.27" layer="95"/>
-<pinref part="C3" gate="C" pin="1"/>
+<pinref part="C3" gate="G$1" pin="1"/>
 </segment>
 </net>
@@
 <segment>
 <pinref part="U2" gate="G$1" pin="V-"/>
-<wire x1="72.39" y1="43.18" x2="77.47" y2="43.18" width="0.1524" layer="91"/>
-<pinref part="C8" gate="C" pin="1"/>
-</segment>
-</net>
+<wire x1="72.39" y1="43.18" x2="78.74" y2="43.18" width="0.1524" layer="91"/>
+<pinref part="C8" gate="G$1" pin="1"/>
+</segment>
+</net>

Commit message: ..
Parts:
- added JP1: JUMPER-SMT_2_NO_SILK_ROUND, SparkFun-Jumpers:JUMPER-SMT_2_NO_SILK_ROUND
Connections:
- new net M1_E_NC: JP1.1, U8.B7
- net M1_E: now also JP1.2; no longer U8.B7
Changed lines of the file:
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@@
 <part name="U$21" library="microbuilder" deviceset="GND" device=""/>
 <part name="U$26" library="microbuilder" deviceset="GND" device=""/>
+<part name="JP1" library="SparkFun-Jumpers" library_urn="urn:adsk.eagle:library:528" deviceset="JUMPER-SMT_2_NO" device="_SILK_ROUND" package3d_urn="urn:adsk.eagle:package:39280/1"/>
 </parts>
 <sheets>
@@
 <attribute name="VALUE" x="178.816" y="134.62" size="1.27" layer="96"/>
 </instance>
+<instance part="JP1" gate="G$1" x="381" y="45.72" smashed="yes">
+<attribute name="NAME" x="381" y="48.514" size="1.778" layer="95" font="vector" align="center"/>
+<attribute name="VALUE" x="381" y="42.926" size="1.778" layer="96" font="vector" align="center"/>
+</instance>
 </instances>
 <busses>
@@
 <net name="M1_E" class="0">
 <segment>
-<pinref part="U8" gate="G$1" pin="B7"/>
-<wire x1="342.9" y1="45.72" x2="360.68" y2="45.72" width="0.1524" layer="91"/>
-<label x="347.98" y="45.72" size="1.778" layer="95"/>
-</segment>
-<segment>
 <wire x1="116.84" y1="71.12" x2="100.33" y2="71.12" width="0.1524" layer="91"/>
 <pinref part="HUB75RGB" gate="G$1" pin="8"/>
@@
 <label x="111.76" y="33.02" size="1.778" layer="95"/>
 </segment>
+<segment>
+<pinref part="JP1" gate="G$1" pin="2"/>
+<wire x1="386.08" y1="45.72" x2="406.4" y2="45.72" width="0.1524" layer="91"/>
+<label x="406.4" y="45.72" size="1.778" layer="95" rot="MR0"/>
+</segment>
 </net>
 <net name="M1_LAT" class="0">
@@
 </segment>
 </net>
+<net name="M1_E_NC" class="0">
+<segment>
+<pinref part="U8" gate="G$1" pin="B7"/>
+<wire x1="342.9" y1="45.72" x2="375.92" y2="45.72" width="0.1524" layer="91"/>
+<label x="347.98" y="45.72" size="1.778" layer="95"/>
+<pinref part="JP1" gate="G$1" pin="1"/>
+</segment>
+</net>

Commit message: thermals="no"
thermals="no"
Changed lines of the file:
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@@
 </plain>
 <instances>
-<instance part="GND1" gate="1" x="101.6" y="104.14" smashed="yes">
-<attribute name="VALUE" x="99.06" y="101.6" size="1.778" layer="96"/>
+<instance part="GND1" gate="1" x="116.84" y="104.14" smashed="yes">
+<attribute name="VALUE" x="114.3" y="101.6" size="1.778" layer="96"/>
 </instance>
 <instance part="HUB75RGB" gate="G$1" x="95.25" y="71.12" smashed="yes" rot="R270">
