File: PCB1/PCB1a_ESP32-DevKitC/PCB1a_ESP32-DevKitC.brd (EAGLE design)
At the start: 125.6 x 84.2 mm, 28 parts, among them J1 691357310006B, J2 618009231421, J5 61004021821, J6 61004021821, U2 MAX232D, U4 TLE9250VSJ, U8 74AHCT245, U9 74AHCT245

Commit message: ..
Routing:
- net B1_3V: track 5.20 -> 31.5 mm, vias 0 -> 2
- net R2_3V: track 11.5 -> 30.8 mm, vias 0 -> 2
- net G1_3V: track 5.20 -> 16.3 mm
- net ADDRB_3V: track 50.7 -> 57.5 mm
- net ADDRC_3V: track 38.9 -> 44.2 mm
- net ADDRA_3V: track 39.0 -> 43.8 mm
- net ADDRD_3V: track 46.1 -> 49.2 mm
- net G2_3V: track 11.8 -> 14.4 mm
- net M1_R1: track 124.3 -> 126.3 mm
- net R1_3V: track 14.1 -> 13.1 mm
- net M1_G1: track 122.7 -> 123.5 mm
- net GND: track 55.2 -> 55.6 mm, vias 467 -> 481
- net B2_3V: vias 0 -> 1

Commit message: thermals="no"/>
thermals="no"/>
Routing:
- net GND: vias 481 -> 482
Changed lines of the file:
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@@
 <drawing>
 <settings>
-<setting alwaysvectorfont="yes"/>
+<setting alwaysvectorfont="no"/>
 <setting verticaltext="up"/>
 </settings>
@@
 <via x="-15.24" y="-26.67" extent="1-16" drill="0.35"/>
 <via x="-26.67" y="-27.94" extent="1-16" drill="0.35"/>
+<via x="-36.83" y="39.37" extent="1-16" drill="0.35"/>
 </signal>
 <signal name="+5V" class="3">

Commit message: Go Production
Parts:
- moved C17 4.49 mm to (17.4, -13.7)
- moved C19 4.49 mm to (23.8, -17.5)
- moved U4 4.49 mm to (22.2, -13.7)
Connections:
- net N$1 renamed 0
- net N$10 renamed VP
- net N$11 renamed 34
- net N$13 renamed EN
- net N$14 renamed USB_TX
- net N$15 renamed USB_RX
- net N$16 renamed 17
- net N$17 renamed 16
- net N$2 renamed CMD
- net N$3 renamed D3
- net N$5 renamed D2
- net N$6 renamed CLK
- net N$7 renamed D0
- net N$8 renamed D1
- net N$9 renamed VN
- removed net B2_3V: J5.19, J5.20, U9.7
- removed net G2_3V: J6.23, J6.24, U9.5
- removed net M1_B2: HUB75RGB..7, HUB75RGB.7, U9.13
- removed net M1_G2: HUB08RG.12, HUB75RGB..6, HUB75RGB.6, U9.15
- removed net M1_R2: HUB08RG.11, HUB75RGB..5, HUB75RGB.5, U9.14
- removed net N$12: J5.1, J5.2
- removed net N$18: J6.1, J6.2
- removed net N$4: J5.3, J5.4
- removed net R2_3V: J6.19, J6.20, U9.6
- new net B0_3V: J6.17, J6.18, U9.4
- new net G0_3V: J6.25, J6.26, U9.3
- new net M1_B0: HUB75RGB..3, HUB75RGB.3, U9.16
- new net M1_G0: HUB08RG.10, HUB12RG.14, HUB75RGB..2, HUB75RGB.2, U9.17
- new net M1_R0: HUB08RG.9, HUB12RG.12, HUB75RGB..1, HUB75RGB.1, U9.18
- new net R0_3V: J6.27, J6.28, U9.2
- net B1_3V: now also J5.19, J5.20, U9.7; no longer J6.17, J6.18, U9.4
- net G1_3V: now also J6.23, J6.24, U9.5; no longer J6.25, J6.26, U9.3
- net GND: now also J5.1, J5.2, J5.3, J5.4, J6.1, J6.2
- net M1_B1: now also HUB75RGB..7, HUB75RGB.7, U9.13; no longer HUB75RGB..3, HUB75RGB.3, U9.16
- net M1_G1: now also HUB08RG.12, HUB75RGB..6, HUB75RGB.6, U9.15; no longer HUB08RG.10, HUB12RG.14, HUB75RGB..2, HUB75RGB.2, U9.17
- net M1_R1: now also HUB08RG.11, HUB75RGB..5, HUB75RGB.5, U9.14; no longer HUB08RG.9, HUB12RG.12, HUB75RGB..1, HUB75RGB.1, U9.18
- net R1_3V: now also J6.19, J6.20, U9.6; no longer J6.27, J6.28, U9.2
Routing:
- net M1_R0: track 0.00 -> 126.3 mm, vias 0 -> 6
- net M1_G0: track 0.00 -> 123.5 mm, vias 0 -> 6
- net M1_G2: track 93.5 -> 0.00 mm, vias 4 -> 0
- net M1_R2: track 90.0 -> 0.00 mm, vias 4 -> 0
- net M1_B0: track 0.00 -> 55.0 mm, vias 0 -> 2
- net M1_B2: track 45.9 -> 0.00 mm, vias 2 -> 0
- net B2_3V: track 44.6 -> 0.00 mm, vias 1 -> 0
- net M1_R1: track 126.3 -> 90.0 mm, vias 6 -> 4
- net B0_3V: track 0.00 -> 31.5 mm, vias 0 -> 2
- net R2_3V: track 30.8 -> 0.00 mm, vias 2 -> 0
- net M1_G1: track 123.5 -> 93.5 mm, vias 6 -> 4
- net +3V3: track 118.6 -> 138.2 mm, vias 3 -> 4
- net R1_3V: track 13.1 -> 30.8 mm, vias 0 -> 2
- net G0_3V: track 0.00 -> 16.3 mm
- net G2_3V: track 14.4 -> 0.00 mm
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Other:
- board text added: "+5V"
- board text added: "0"
- board text added: "1"
- board text added: "12"
- board text added: "13"
- board text added: "14"
- board text added: "15"
- board text added: "16"
- board text added: "17"
- board text added: "18"
- board text added: "19"
- board text added: "2"
- board text added: "21"
- board text added: "22"
- board text added: "23"
- board text added: "25"
- board text added: "26"
- board text added: "27"
- board text added: "32"
- board text added: "33"
- board text added: "34"
- board text added: "35"
- board text added: "3V3"
- board text added: "4"
- board text added: "5"
- board text added: "6"
- board text added: "9"
- board text added: "CAN1 RXD"
- board text added: "CAN1 TXD"
- board text added: "CLK"
- board text added: "CMD"
- board text added: "D0"
- board text added: "D1"
- board text added: "D2"
- board text added: "D3"
- board text added: "E"
- board text added: "EN"
- board text added: "H"
- board text added: "L"
- board text added: "LAT"
- board text added: "RS232 RXD"
- board text added: "RS232 TXD"
- board text added: "RX"
- board text added: "TX"
- board text added: "VP"
