File: PCB1/PCB1a_T-ETH-Lite-ESP32S3/PCB1a_T-ETH-Lite-ESP32S3.sch (EAGLE design)
At the start: 42 parts, among them J1 691357310006B, J2 618009231421, J5 61004021821, J6 61004021821, U2 MAX232D, U4 TLE9250VSJ, U8 74AHCT245, U9 74AHCT245

Commit message: ..
Parts:
- added J3: 61003221821, Wurth_Connectors_WR-PHD:6100XX21821_61003221821
- added J4: 61003021821, Wurth_Connectors_WR-PHD:6100XX21821_61003021821
Connections:
- net +5V: now also J3.1, J3.2
- net GND: now also J3.3, J3.4
Changed lines of the file:
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@@
 <part name="GND3" library="supply1" deviceset="GND" device=""/>
 <part name="GND6" library="supply1" deviceset="GND" device=""/>
+<part name="J3" library="Wurth_Connectors_WR-PHD" library_urn="urn:adsk.eagle:library:14804658" deviceset="6100XX21821_61003221821" device="" package3d_urn="urn:adsk.eagle:package:14805694/2" value=" 61003221821 "/>
+<part name="J4" library="Wurth_Connectors_WR-PHD" library_urn="urn:adsk.eagle:library:14804658" deviceset="6100XX21821_61003021821" device="" package3d_urn="urn:adsk.eagle:package:14805693/2" value=" 61003021821 "/>
+<part name="P+5" library="supply1" library_urn="urn:adsk.eagle:library:371" deviceset="+5V" device=""/>
+<part name="GND24" library="supply1" deviceset="GND" device=""/>
 </parts>
 <sheets>
@@
 <attribute name="VALUE" x="241.3" y="-35.56" size="1.778" layer="96" rot="R180"/>
 </instance>
+<instance part="J3" gate="G$1" x="274.32" y="-157.48" smashed="yes" rot="R270">
+<attribute name="NAME" x="275.398" y="-137.36" size="1.016" layer="95" rot="R270" align="bottom-right"/>
+<attribute name="VALUE" x="272.74" y="-137.41" size="1.016" layer="96" rot="R270" align="bottom-right"/>
+</instance>
+<instance part="J4" gate="G$1" x="254" y="-157.48" smashed="yes" rot="R270">
+<attribute name="NAME" x="255.078" y="-137.36" size="1.016" layer="95" rot="R270" align="bottom-right"/>
+<attribute name="VALUE" x="252.42" y="-137.41" size="1.016" layer="96" rot="R270" align="bottom-right"/>
+</instance>
+<instance part="P+5" gate="1" x="289.56" y="-129.54" smashed="yes" rot="MR0">
+<attribute name="VALUE" x="289.56" y="-127" size="1.778" layer="96" rot="MR0"/>
+</instance>
+<instance part="GND24" gate="1" x="309.88" y="-147.32" smashed="yes">
+<attribute name="VALUE" x="307.34" y="-149.86" size="1.778" layer="96"/>
+</instance>
 </instances>
 <busses>
@@
 <label x="248.92" y="-88.9" size="1.778" layer="95"/>
 </segment>
+<segment>
+<pinref part="J3" gate="G$1" pin="2"/>
+<pinref part="J3" gate="G$1" pin="1"/>
+<wire x1="269.24" y1="-139.7" x2="279.4" y2="-139.7" width="0.1524" layer="91"/>
+<pinref part="P+5" gate="1" pin="+5V"/>
+<wire x1="279.4" y1="-139.7" x2="289.56" y2="-139.7" width="0.1524" layer="91"/>
+<wire x1="289.56" y1="-139.7" x2="289.56" y2="-132.08" width="0.1524" layer="91"/>
+<junction x="279.4" y="-139.7"/>
+</segment>
 </net>
 <net name="GND" class="0">
@@
 <junction x="294.64" y="-43.18"/>
 </segment>
+<segment>
+<pinref part="J3" gate="G$1" pin="4"/>
+<pinref part="J3" gate="G$1" pin="3"/>
+<wire x1="269.24" y1="-142.24" x2="279.4" y2="-142.24" width="0.1524" layer="91"/>
+<pinref part="GND24" gate="1" pin="GND"/>
+<wire x1="309.88" y1="-144.78" x2="309.88" y2="-142.24" width="0.1524" layer="91"/>
+<wire x1="309.88" y1="-142.24" x2="279.4" y2="-142.24" width="0.1524" layer="91"/>
+<junction x="279.4" y="-142.24"/>
+</segment>
 </net>
