File: Ethernet/Teensy/Teensy_ETH/Teensy_ETH.brd (EAGLE design)
At the start: 160 x 100 mm, 3 parts, among them M1 TEENSY4.1

Commit message: sicherung
Parts:
- added C1, C2: 100000pF, Wurth_Capacitors_WCAP-CSST:WCAP-CSST_0603_R
- added C3, C4: 1000pF, Wurth_Capacitors_WCAP-CSMH:WCAP-CSMH_1206_H1.6_R
- added D1, D2: 3.3Vdc, Wurth_EMC Components_WE-TVS:WE-TVS_DFN1210-6L
- added J1: 615008137421, Wurth_Connectors_WR-MJ:615008137421
- added L1, L2: 260Ohm@ 100 MHz, Wurth_EMC Components_WE-CNSW:WE-CNSW_0805
- added R1, R2, R3, R4: RES, 75.0, 1%, 0.125 W, AECQ200 Grade 0, 0805, resistor:R0805
- moved T1 88.9 mm to (133.3, 30.5), turned to 270 degrees
- moved T2 82.9 mm to (128.3, 30.5), turned to 270 degrees
- moved M1 41.8 mm to (114.3, 62.9), turned to 180 degrees
Connections:
- new net ER_N: M1.ER-, T2.1
- new net ER_P: M1.ER+, T2.2
- new net ET_N: M1.ET+, T1.1
- new net ET_P: M1.ET-, T1.2
- new net FR_N: L2.4, T2.6
- new net FR_P: L2.1, T2.7
- new net FT_N: L1.4, T1.6
- new net FT_P: L1.1, T1.7
- new net N$17: C1.2, T1.5
- new net N$18: C2.2, T2.5
- new net N$19: C3.2, R1.1, R2.1, R3.1, R4.1
- new net N$7: J1.4, J1.5, R3.2
- new net N$8: J1.7, J1.8, R4.2
- new net PE: C3.1, C4.1, D1.3, D2.3, J1.S1, J1.S2
- new net R_N: D2.2, J1.6, L2.3
- new net R_P: D2.1, J1.3, L2.2
- new net T_N: D1.1, J1.2, L1.3
- new net T_P: D1.2, J1.1, L1.2
- new net V-: C1.1, C2.1, C4.2
- net N$1: now also R2.2
- net N$2: now also R1.2
Routing:
- net N$19: track 0.00 -> 33.6 mm
- net ET_N: track 0.00 -> 32.6 mm
- net ET_P: track 0.00 -> 32.3 mm
- net ER_P: track 0.00 -> 26.4 mm
- net ER_N: track 0.00 -> 26.4 mm
- net N$7: track 0.00 -> 24.0 mm
- net N$1: track 0.00 -> 22.8 mm
- net R_P: track 0.00 -> 17.8 mm, vias 0 -> 2
- net N$8: track 0.00 -> 17.0 mm
- net T_N: track 0.00 -> 16.9 mm, vias 0 -> 2
- net N$2: track 0.00 -> 16.1 mm
- net T_P: track 0.00 -> 15.7 mm
- net R_N: track 0.00 -> 13.3 mm
- net FR_P: track 0.00 -> 5.06 mm
- net FT_P: track 0.00 -> 5.06 mm
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- added copper zone on layer 1, net PE
- added copper zone on layer 1, net V-
