File: Ethernet/Teensy/Teensy_ETH/Teensy_ETH.sch (EAGLE design)
At the start: 1 part, among them M1 TEENSY4.1

Commit message: 1st Version with WE WE-STST 74930000
WE-STST 74930000
Parts:
- added T1, T2: (no value), Wurth_Signal & Communications_WE-STST:WE-STST_4532_74930000
Connections:
- new net N$1: T1.3, T1.4
- new net N$2: T2.3, T2.4
Changed lines of the file:
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@@
 <parts>
 <part name="M1" library="teensy4.1.dist" deviceset="TEENSY4.1" device=""/>
+<part name="T1" library="Wurth_Signal &amp; Communications_WE-STST" library_urn="urn:adsk.eagle:library:14998825" deviceset="WE-STST_4532" device="_74930000" package3d_urn="urn:adsk.eagle:package:14998834/5"/>
+<part name="T2" library="Wurth_Signal &amp; Communications_WE-STST" library_urn="urn:adsk.eagle:library:14998825" deviceset="WE-STST_4532" device="_74930000" package3d_urn="urn:adsk.eagle:package:14998834/5"/>
 </parts>
 <sheets>
@@
 <instance part="M1" gate="G$2" x="48.26" y="83.82" smashed="yes">
 <attribute name="NAME" x="43.18" y="91.948" size="1.27" layer="95" font="vector"/>
-</instance>
-<instance part="M1" gate="G$3" x="78.74" y="86.36" smashed="yes">
-<attribute name="NAME" x="73.66" y="94.488" size="1.27" layer="94" font="vector"/>
 </instance>
 <instance part="M1" gate="G$1" x="114.3" y="73.66" smashed="yes">
@@
 </nets>
 </sheet>
+<sheet>
+<plain>
+</plain>
+<instances>
+<instance part="M1" gate="G$3" x="25.4" y="68.58" smashed="yes" rot="R180">
+<attribute name="NAME" x="30.48" y="60.452" size="1.27" layer="94" font="vector" rot="R180"/>
+</instance>
+<instance part="T1" gate="G$1" x="111.76" y="101.6" smashed="yes">
+<attribute name="NAME" x="111.76" y="115.27" size="1.778" layer="95" align="bottom-center"/>
+<attribute name="VALUE" x="106.68" y="85.09" size="1.778" layer="96"/>
+</instance>
+<instance part="T2" gate="G$1" x="111.76" y="63.5" smashed="yes">
+<attribute name="NAME" x="111.76" y="77.17" size="1.778" layer="95" align="bottom-center"/>
+<attribute name="VALUE" x="106.68" y="46.99" size="1.778" layer="96"/>
+</instance>
+</instances>
+<busses>
+</busses>
+<nets>
+<net name="N$1" class="0">
+<segment>
+<pinref part="T1" gate="G$1" pin="4"/>
+<pinref part="T1" gate="G$1" pin="3"/>
+<wire x1="119.38" y1="104.14" x2="119.38" y2="99.06" width="0.1524" layer="91"/>
+</segment>
+</net>
+<net name="N$2" class="0">
+<segment>
+<pinref part="T2" gate="G$1" pin="4"/>
+<pinref part="T2" gate="G$1" pin="3"/>
+<wire x1="119.38" y1="66.04" x2="119.38" y2="60.96" width="0.1524" layer="91"/>
+</segment>
+</net>
+</nets>
+</sheet>
 </sheets>
 </schematic>
 </drawing>
+<compatibility>
+<note version="8.2" severity="warning">
+Since Version 8.2, EAGLE supports online libraries. The ids
+of those online libraries will not be understood (or retained)
+with this version.
+</note>
+<note version="8.3" severity="warning">
+Since Version 8.3, EAGLE supports URNs for individual library
+assets (packages, symbols, and devices). The URNs of those assets
+will not be understood (or retained) with this version.
+</note>
+<note version="8.3" severity="warning">
+Since Version 8.3, EAGLE supports the association of 3D packages
+with devices in libraries, schematics, and board files. Those 3D
+packages will not be understood (or retained) with this version.
+</note>
+</compatibility>
 </eagle>

Commit message: sicherung
Parts:
- added C1, C2: 100000pF, Wurth_Capacitors_WCAP-CSST:WCAP-CSST_0603_885382206004_R
- added C3, C4: 1000pF, Wurth_Capacitors_WCAP-CSMH:WCAP-CSMH_1206_H1.6_885342208024
- added D1, D2: 3.3Vdc, Wurth_EMC Components_WE-TVS:WE-TVS-SS_DFN1210-6L_824012823
- added J1: 615008137421, Wurth_Connectors_WR-MJ:615008137421
- added L1, L2: 260Ohm@ 100 MHz, Wurth_EMC Components_WE-CNSW:WE-CNSW_0805_744231261
- added R1, R2, R3, R4: RES, 75.0, 1%, 0.125 W, AECQ200 Grade 0, 0805, resistor:R-EU_R0805
Connections:
- new net ER_N: M1G$3.ER-, T2.1
- new net ER_P: M1G$3.ER+, T2.2
- new net ET_N: M1G$3.ET-, T1.1
- new net ET_P: M1G$3.ET+, T1.2
- new net FR_N: L2.1, T2.6
- new net FR_P: L2.4, T2.7
- new net FT_N: L1.1, T1.6
- new net FT_P: L1.4, T1.7
- new net N$17: C1.2, T1.5
- new net N$18: C2.2, T2.5
- new net N$19: C3.2, R1.1, R2.1, R3.1, R4.1
- new net N$7: J1.4, J1.5, R3.2
- new net N$8: J1.7, J1.8, R4.2
- new net PE: C3.1, C4.1, D1.GND, D2.GND, J1.SHIELD
- new net R_N: D2.I/O2, J1.6, L2.2
- new net R_P: D2.I/O1, J1.3, L2.3
- new net T_N: D1.I/O1, J1.2, L1.2
- new net T_P: D1.I/O2, J1.1, L1.3
- new net V-: C1.1, C2.1, C4.2
- net N$1: now also R2.2
- net N$2: now also R1.2
Other:
- moved on the sheet: M1G$3, T1, T2
