File: PCB1/PCB1a_Adapter/PCB1a_Adapter.sch (EAGLE design)
At the start: 42 parts, among them J1 691357310006B, J2 618009231421, J5 61004021821, J6 61004021821, U2 MAX232D, U4 TLE9250VSJ, U8 74AHCT245, U9 74AHCT245

Commit message: Update PCB design settings and connector library description.
- Update PCB design settings for vector font to "alwaysvectorfont=yes" and vertical text to "up".
- Remove specific library references from the PCB design file.
- Modify a connector library description in the board file.
Parts:
- removed C1: 470uF, Wurth_Capacitors_WCAP-AS5H:WCAP-AS5H_10X10.5_865230357008
- removed C15: 47nF, Wurth_Capacitors_WCAP-CSGP:WCAP-CSGP_0805_H0.8_885012207096_50V(DC)_R
- removed C17, C19, C2, C3, C4, C5, C6, C7, C8: 100nF, Wurth_Capacitors_WCAP-CSGP:WCAP-CSGP_0805_H0.8_885012207098_50V(DC)_R
- removed D1: 5V, Wurth_EMC Components_WE-TVSP:WE-TVSP_DO-214AB_3000W_BI_824551500
- removed D11: 24Vdc, Wurth_EMC Components_WE-TVS:WE-TVS_SOT23-3L_824094024
- removed J1: 691357310006B, Wurth_Connectors_WR-TBL Pluggable Connector:691357310006B
- removed J2: 618009231421, Wurth_Connectors_WR-DSUB:6180XX231421_618009231421
- removed J5, J6: 61004021821, Wurth_Connectors_WR-PHD:6100XX21821_61004021821
- removed JP1: JUMPER-SMT_2_NO_SILK_ROUND, SparkFun-Jumpers:JUMPER-SMT_2_NO_SILK_ROUND
- removed R1, R3: 60R, resistor:R-EU_R0805
- removed U$10, U$11, U$13, U$15, U$16, U$17, U$2, U$3, U$4, U$5, U$6, U$7, U$8, U$9: NC, eclibrary:NC
- removed U2: MAX232D, IC:MAX3232-SOIC16
- removed U4: TLE9250VSJ, TLE9250VSJ:TLE9250VSJ
- removed U8, U9: 74AHCT245, microbuilder:74LCX245_TSSOP20
Connections:
- removed net +3V3: C19.1, C3.1, C4.2, J6.3, J6.4, U2.VCC, U4.VIO
- removed net +5V: C1.+, C17.1, C2.2, C5.2, D1.2, J1.3, J6.39, J6.40, U4.VCC, U8.T/R, U8.VCC, U9.T/R, U9.VCC
- removed net 0: J5.29, J5.30
- removed net 16: J5.25, J5.26, U$17.P$1
- removed net 17: J5.23, J5.24, U$16.P$1
- removed net 232_RX: J2.2, U2.RIN1
- removed net 232_TX: J2.3, U2.DOUT1
- removed net 34: J6.11, J6.12, U$10.P$1
- removed net ADDRA_3V: J5.17, J5.18, U8.A4
- removed net ADDRB_3V: J5.7, J5.8, U9.A8
- removed net ADDRC_3V: J5.13, J5.14, U8.A5
- removed net ADDRD_3V: J5.27, J5.28, U8.A3
- removed net ADDRE_3V: J6.21, J6.22, U8.A7
- removed net B0_3V: J6.17, J6.18, U9.A3
- removed net B1_3V: J5.19, J5.20, U9.A6
- removed net CAN1_RXD: J6.13, J6.14, U4.RXD
- removed net CAN1_TXD: J5.21, J5.22, U4.TXD
- removed net CAN_N: D11.I/O1, J1.5, R3.2, U4.CANL
- removed net CAN_P: D11.I/O2, J1.6, R1.2, U4.CANH
- removed net CLK: J5.39, J5.40, U$5.P$1
- removed net CLK_3V: J5.31, J5.32, U9.A7
- removed net CMD: J6.37, J6.38, U$2.P$1
- removed net D0: J5.37, J5.38, U$6.P$1
- removed net D1: J5.35, J5.36, U$7.P$1
- removed net D2: J6.33, J6.34, U$4.P$1
- removed net D3: J6.35, J6.36, U$3.P$1
- removed net EN: J6.5, J6.6, U$11.P$1
- removed net G0_3V: J6.25, J6.26, U9.A2
- removed net G1_3V: J6.23, J6.24, U9.A4
- removed net LAT_3V: J5.33, J5.34, U8.A6
- removed net M1_E_NC: JP1.1, U8.B7
- removed net N$20: C15.1, R1.1, R3.1
- removed net N$33: C6.2, U2.C1+
- removed net N$34: C6.1, U2.C1-
- removed net N$35: C7.2, U2.C2+
- removed net N$36: C7.1, U2.C2-
- removed net N$37: C4.1, U2.V+
- removed net N$38: C8.1, U2.V-
- removed net N$39: U2.ROUT2
- removed net N$40: U2.DIN2
- removed net N$46: U2.DOUT2
- removed net N$47: U2.RIN2
- removed net OE_3V: J6.31, J6.32, U8.A8
- removed net R0_3V: J6.27, J6.28, U9.A1
- removed net R1_3V: J6.19, J6.20, U9.A5
- removed net RX: J6.15, J6.16, U2.ROUT1
- removed net TX: J5.5, J5.6, U2.DIN1
- removed net USB_RX: J5.11, J5.12, U$15.P$1
- removed net USB_TX: J5.10, J5.9, U$13.P$1
- removed net VN: J6.10, J6.9, U$8.P$1
- removed net VP: J6.7, J6.8, U$9.P$1
- net GND: no longer C1.-, C15.2, C17.2, C19.2, C2.1, C3.2, C5.1, C8.2, D1.1, D11.GND, J1.1, J1.4, J2.5, J2.SHIELD, J5.1, J5.15, J5.16, J5.2, J5.3, J5.4, J6.1, J6.2, J6.29, J6.30, U2.GND, U4.GND, U4.NEN, U8./OE, U8.A1, U8.A2, U8.GND, U9./OE, U9.GND
- net M1_A: no longer U8.B4
- net M1_B: no longer U9.B8
- net M1_B0: no longer U9.B3
- net M1_B1: no longer U9.B6
- net M1_C: no longer U8.B5
- net M1_CLK: no longer U9.B7
- net M1_D: no longer U8.B3
- net M1_E: no longer JP1.2
- net M1_G0: no longer U9.B2
- net M1_G1: no longer U9.B4
- net M1_LAT: no longer U8.B6
- net M1_OE: no longer U8.B8
- net M1_R0: no longer U9.B1
- net M1_R1: no longer U9.B5
Other:
- note removed: "All pins marked with X are unused by SmartLED Library"
- note removed: "ESP32"
- note removed: "Free: Input/Analog Only"
- note removed: "LEVEL SHIFTERS"
- note removed: "MatrixHardware: Hub75 Adapter Pinout, but G2 on 27"
- note removed: "NC on WROVER"
- note removed: "RESERVED FOR FLASH"
- note removed: "RESET"
- note removed: "USB Comms"
- note removed: "Very low electromagnetic emission (EME) allows the use without additional common mode choke TLE9250VSJ"
